Commit message: changed robot design and launch paramaters

File: udacity_bot/urdf/udacity_bot.xacro (robot description, xacro)
@@ -1,11 +1,12 @@
 <?xml version='1.0'?>
 <robot name="udacity_bot" xmlns:xacro="http://www.ros.org/wiki/xacro">
-  <xacro:include filename="$(find udacity_bot)/urdf/udacity_bot.gazebo" />
+  <xacro:include filename="$(find udacity_bot)/urdf/udacity_bot.gazebo"/>
   <link name="robot_footprint"></link>
   <joint name="robot_footprint_joint" type="fixed">
-    <origin xyz="0 0 0" rpy="0 0 0" />
+    <origin xyz="0 0 0" rpy="0 0 0"/>
     <parent link="robot_footprint"/>
-    <child link="chassis" />
-  </joint>
+    <child link="chassis"/>
+  </joint>
+  <!-- Left wheel -->
   <joint type="continuous" name="left_wheel_hinge">
     <origin xyz="0 0.15 0" rpy="0 0 0"/>
@@ -29,5 +30,5 @@
       <origin xyz="0 0 0" rpy=" 0 1.5707 1.5707"/>
       <geometry>
-        <cylinder radius="0.1" length="0.05"/>
+        <cylinder radius="0.05" length="0.05"/>
       </geometry>
     </collision>
@@ -35,8 +36,9 @@
       <origin xyz="0 0 0" rpy=" 0 1.5707 1.5707"/>
       <geometry>
-        <cylinder radius="0.1" length="0.05"/>
-      </geometry>
-    </visual>
-  </link>
+        <cylinder radius="0.05" length="0.05"/>
+      </geometry>
+    </visual>
+  </link>
+  <!-- Right wheel -->
   <joint type="continuous" name="right_wheel_hinge">
     <origin xyz="0 -0.15 0" rpy="0 0 0"/>
@@ -60,5 +62,5 @@
       <origin xyz="0 0 0" rpy=" 0 1.5707 1.5707"/>
       <geometry>
-        <cylinder radius="0.1" length="0.05"/>
+        <cylinder radius="0.05" length="0.05"/>
       </geometry>
     </collision>
@@ -66,10 +68,11 @@
       <origin xyz="0 0 0" rpy=" 0 1.5707 1.5707"/>
       <geometry>
-        <cylinder radius="0.1" length="0.05"/>
-      </geometry>
-    </visual>
-  </link>
+        <cylinder radius="0.05" length="0.05"/>
+      </geometry>
+    </visual>
+  </link>
+  <!-- Camera -->
   <joint type="fixed" name="camera_joint">
-    <origin xyz="0.2 0 0" rpy="0 0 0"/>
+    <origin xyz="0.275 0 0.1" rpy="0 0 0"/>
     <child link="camera"/>
     <parent link="chassis"/>
@@ -98,6 +101,7 @@
     </visual>
   </link>
+  <!-- Laser scanner -->
   <joint type="fixed" name="hokuyo_joint">
-    <origin xyz="0.15 0 0.1" rpy="0 0 0"/>
+    <origin xyz="0 0 0.20" rpy="0 0 0"/>
     <child link="hokuyo"/>
     <parent link="chassis"/>
@@ -126,4 +130,5 @@
     </visual>
   </link>
+  <!-- Chassis -->
   <link name='chassis'>
     <pose>0 0 0.1 0 0 0</pose>
@@ -137,38 +142,62 @@
       />
     </inertial>
-    <collision name='collision'>
-      <origin xyz="0 0 0" rpy=" 0 0 0"/>
-      <geometry>
-        <box size=".4 .2 .1"/>
+    <!--<collision name='collision'>-->
+    <!--<origin xyz="0 0 0" rpy=" 0 0 0"/>-->
+    <!--<geometry>-->
+    <!--<box size=".4 .2 .1"/>-->
+    <!--</geometry>-->
+    <!--</collision>-->
+    <!--<visual name='chassis_visual'>-->
+    <!--<origin xyz="0 0 0" rpy=" 0 0 0"/>-->
+    <!--<geometry>-->
+    <!--<box size=".4 .2 .1"/>-->
+    <!--</geometry>-->
+    <!--</visual>-->
+    <collision name='chassis_collision'>
+      <origin xyz="0 0 0.05" rpy=" 0 0 0"/>
+      <geometry>
+        <cylinder radius="0.25" length="0.15"/>
       </geometry>
     </collision>
     <visual name='chassis_visual'>
-      <origin xyz="0 0 0" rpy=" 0 0 0"/>
-      <geometry>
-        <box size=".4 .2 .1"/>
+      <origin xyz="0 0 0.05" rpy=" 0 0 0"/>
+      <geometry>
+        <cylinder radius="0.25" length="0.15"/>
+      </geometry>
+    </visual>
+    <collision name='chassis_dome_collision'>
+      <origin xyz="0 0 0.1125" rpy=" 0 0 0"/>
+      <geometry>
+        <sphere radius="0.1"/>
+      </geometry>
+    </collision>
+    <visual name='chassis_dome_visual'>
+      <origin xyz="0 0 0.1125" rpy=" 0 0 0"/>
+      <geometry>
+        <sphere radius="0.1"/>
       </geometry>
     </visual>
     <collision name='back_caster_collision'>
-      <origin xyz="-0.15 0 -0.05" rpy=" 0 0 0"/>
-      <geometry>
-        <sphere radius="0.0499"/>
+      <origin xyz="-0.15 0 -0.025" rpy=" 0 0 0"/>
+      <geometry>
+        <sphere radius="0.02499"/>
       </geometry>
     </collision>
     <visual name='back_caster_visual'>
-      <origin xyz="-0.15 0 -0.05" rpy=" 0 0 0"/>
-      <geometry>
-        <sphere radius="0.05"/>
+      <origin xyz="-0.15 0 -0.025" rpy=" 0 0 0"/>
+      <geometry>
+        <sphere radius="0.025"/>
       </geometry>
     </visual>
     <collision name='front_caster_collision'>
-      <origin xyz="0.15 0 -0.05" rpy=" 0 0 0"/>
-      <geometry>
-        <sphere radius="0.0499"/>
+      <origin xyz="0.15 0 -0.025" rpy=" 0 0 0"/>
+      <geometry>
+        <sphere radius="0.02499"/>
       </geometry>
     </collision>
     <visual name='front_caster_visual'>
-      <origin xyz="0.15 0 -0.05" rpy=" 0 0 0"/>
-      <geometry>
-        <sphere radius="0.05"/>
+      <origin xyz="0.15 0 -0.025" rpy=" 0 0 0"/>
+      <geometry>
+        <sphere radius="0.025"/>
       </geometry>
     </visual>
